File: EAGLE/GPS_radiologger_v2_energy_harvesting.brd (EAGLE design)
At the start: 11.4 x 20.7 mm, 23 parts, among them Q1 1.1A/60V/600mΩ, U2 CC1350F128RGZT, U3 TPL5110, Y3 32.768kHz

Commit message: added v3
Parts:
- removed C11, C22: 8.2 pF, SparkFun-Capacitors:0402-TIGHT
- removed C12, C14: 4.7 pF, SparkFun-Capacitors:0402-TIGHT
- removed C13, C3, C4: 12 pF, SparkFun-Capacitors:0402-TIGHT
- removed C15, C21: 330 pF, SparkFun-Capacitors:0402-TIGHT
- removed J1: (no value), SparkFun-Connectors:1X01_OFFSET
- removed L11: 33 nH, SparkFun-Coils:0402_MURATA
- removed L12, L21: 15 nH, SparkFun-Coils:0402_MURATA
- removed L13, L14: 20 nH, SparkFun-Coils:0402_MURATA
- removed R1: 100K, SparkFun-Resistors:0402
- removed U$1, U$2: TRISOLX_8X16, TrisolX_Solar_Cells:TRISOLX_8X16
- removed U$3: 2.4 pF, SparkFun-Capacitors:0402_MURATA
- removed U2: CC1350F128RGZT, CC1350F128RGZT:RGZ48
- removed Y3: 32.768kHz, SparkFun-Clocks:CRYSTAL-SMD-3.2X1.5MM
Connections:
- removed net N$10: C15.2, J1.1
- removed net N$11: C3.1, U2.4, Y3.P$1
- removed net N$12: C4.1, U2.5, Y3.P$2
- removed net N$13: R1.1, U$3.P$1, U2.35
- removed net N$7: C13.1, L13.P$2, L14.P$1
- removed net N$8: C14.1, C15.1, L14.P$2
- removed net N$9: C12.1, C22.1, L12.P$2, L13.P$1
- removed net RF_N: C22.2, L11.P$2, L21.P$2, U2.2
- removed net RF_P: C11.1, L11.P$1, L12.P$1, U2.1
- removed net RX_TX: C21.1, L21.P$1, U2.3
- removed net SCL: U2.9
- removed net SDA: U2.10
- removed net VDDR: U2.45
- removed net VDDR_RF: U2.48
- removed net VDDS: U2.44
- removed net VDDS2: U2.13
- removed net VDDS3: U2.22
- removed net VDDS_DCDC: U2.34
- net DONE: no longer U2.11
- net GND: no longer C11.2, C12.2, C13.2, C14.2, C21.2, C3.2, C4.2, U$3.P$2
