File: EAGLE/GPS_radiologger_v2_energy_harvesting.sch (EAGLE design)
At the start: 23 parts, among them Q1 1.1A/60V/600mΩ, U2 CC1350F128RGZT, U3 TPL5110, Y3 32.768kHz

Commit message: added v3
Parts:
- removed C11, C22: 8.2 pF, SparkFun-Capacitors:0.1UF-0402T-16V-10%
- removed C12, C14: 4.7 pF, SparkFun-Capacitors:0.1UF-0402T-16V-10%
- removed C13, C3, C4: 12 pF, SparkFun-Capacitors:0.1UF-0402T-16V-10%
- removed C15, C21: 330 pF, SparkFun-Capacitors:0.1UF-0402T-16V-10%
- removed J1: (no value), SparkFun-Connectors:CONN_01OFFSET
- removed L11: 33 nH, SparkFun-Coils:19NH-0402
- removed L12, L21: 15 nH, SparkFun-Coils:19NH-0402
- removed L13, L14: 20 nH, SparkFun-Coils:19NH-0402
- removed R1: 100K, SparkFun-Resistors:100KOHM-0402-1/16W-1%
- removed U$1, U$2: TRISOLX_8X16, TrisolX_Solar_Cells:TRISOLX_8X16
- removed U$3: 2.4 pF, SparkFun-Capacitors:2.4PF-0402
- removed U2: CC1350F128RGZT, CC1350F128RGZT:CC1350F128RGZT
- removed Y3: 32.768kHz, SparkFun-Clocks:CRYSTAL-32.768KHZSMD-3.2X1.5
Connections:
- removed net N$10: C15.2, J1.1
- removed net N$11: C3.1, U2A.X32K_Q1, Y3.1
- removed net N$12: C4.1, U2A.X32K_Q2, Y3.2
- removed net N$13: R1.1, U$3.1, U2A.RESET_N
- removed net N$7: C13.1, L13.2, L14.1
- removed net N$8: C14.1, C15.1, L14.2
- removed net N$9: C12.1, C22.1, L12.2, L13.1
- removed net RF_N: C22.2, L11.2, L21.2, U2A.RF_N
- removed net RF_P: C11.1, L11.1, L12.1, U2A.RF_P
- removed net RX_TX: C21.1, L21.1, U2A.RX_TX
- removed net SCL: U2A.DIO_4
- removed net SDA: U2A.DIO_5
- net DONE: no longer U2A.DIO_6
- net GND: no longer C11.2, C12.2, C13.2, C14.2, C21.2, C3.2, C4.2, U$3.2
Other:
- note added: "868 MHz Matching Network"
- note added: "GNSS Receiver"
- note removed: "! Matching network part numbers match Texas Instruments 433 MHz reference doc SWRC330"
- note removed: "433 MHz Matching Network"
- note removed: "GNSS / GLONASS Receiver"
