File: EAGLE/GPS_radiologger_v3.sch (EAGLE design)
At the start: 22 parts, among them Q1 1.1A/60V/600mΩ, U1 ATSAMD21E18A-U, U3 TPL5110

Commit message: more_pcb_edits
Parts:
- added U2: UBLOX_ZOE_M8Q-0-10, SparkFun-GPS:UBLOX_ZOE_M8Q-0-10
- added U4: RFM95W, SparkFun-RF:RFM95W
Changed lines of the file:
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@@
 <part name="GND4" library="supply1" library_urn="urn:adsk.eagle:library:371" deviceset="GND" device=""/>
 <part name="U1" library="SparkFun-IC-Microcontroller" deviceset="ATSAMD21E18A-U" device=""/>
+<part name="U2" library="SparkFun-GPS" deviceset="UBLOX_ZOE_M8Q-0-10" device=""/>
+<part name="U4" library="SparkFun-RF" deviceset="RFM95W" device=""/>
 </parts>
 <sheets>
@@
 <attribute name="VALUE" x="170.18" y="45.72" size="2.54" layer="96"/>
 </instance>
+<instance part="U2" gate="G$1" x="116.84" y="33.02" smashed="yes">
+<attribute name="NAME" x="101.6" y="60.96" size="2.54" layer="95"/>
+<attribute name="VALUE" x="101.6" y="5.08" size="2.54" layer="96"/>
+</instance>
+<instance part="U4" gate="G$1" x="43.18" y="40.64" smashed="yes">
+<attribute name="NAME" x="30.512" y="58.96" size="1.778" layer="95"/>
+</instance>
 </instances>
