File: EAGLE/GPS_radiologger_v3.brd (EAGLE design)
At the start: 24.6 x 16.5 mm, 22 parts, among them Q1 1.1A/60V/600mΩ, U1 ATSAMD21E18A-U, U3 TPL5110

Commit message: more_pcb_edits
Parts:
- added U2: UBLOX_ZOE_M8Q-0-10, SparkFun-GPS:UBLOX_ZOE_M8-0-10
- added U4: RFM95W, SparkFun-RF:RFM95/96/97/98W
- moved U1 20.5 mm to (4.16, 3.69)
Connections:
- new net VCC: U2.24, U2.25
- new net V_BCKP: U2.16
- new net V_CORE: U2.27
- new net V_DCDC_OUT: U2.26
- net GND: now also U2.1, U2.10, U2.11, U2.12, U2.17, U2.23, U2.3, U2.37, U2.38, U2.39, U2.40, U2.41, U2.44, U2.49, U2.5, U2.7, U2.8, U2.9
Changed lines of the file:
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@@
 <attribute name="VALUE" x="1.621" y="-10.53" size="0.6096" layer="27" font="vector" ratio="20" rot="R90" align="top-center"/>
 </element>
-<element name="U1" library="SparkFun-IC-Microcontroller" package="QFN-32_SAMD" value="ATSAMD21E18A-U" x="-5.87" y="-14.22" smashed="yes">
-<attribute name="NAME" x="-8.36" y="-11.2" size="1" layer="25"/>
-<attribute name="PROD_ID" value="IC-14428" x="-5.87" y="-14.22" size="1.778" layer="27" display="off"/>
-<attribute name="VALUE" x="-8.372" y="-18.224" size="1" layer="27"/>
+<element name="U1" library="SparkFun-IC-Microcontroller" package="QFN-32_SAMD" value="ATSAMD21E18A-U" x="4.16" y="3.69" smashed="yes">
+<attribute name="NAME" x="1.67" y="6.71" size="1" layer="25"/>
+<attribute name="PROD_ID" value="IC-14428" x="4.16" y="3.69" size="1.778" layer="27" display="off"/>
+<attribute name="VALUE" x="1.658" y="-0.314" size="1" layer="27"/>
+</element>
+<element name="U2" library="SparkFun-GPS" package="UBLOX_ZOE_M8-0-10" value="UBLOX_ZOE_M8Q-0-10" x="-9.64" y="2.04" smashed="yes">
+<attribute name="NAME" x="-11.886" y="5.175" size="1" layer="25"/>
+<attribute name="PROD_ID" value="IC-14251" x="-9.64" y="2.04" size="1.778" layer="27" display="off"/>
+<attribute name="VALUE" x="-12.013" y="-1.825" size="1" layer="27"/>
+</element>
+<element name="U4" library="SparkFun-RF" package="RFM95/96/97/98W" value="RFM95W" x="17.16" y="-10.12" smashed="yes" rot="R90">
+<attribute name="PROD_ID" value="IC-13959" x="17.16" y="-10.12" size="1.778" layer="27" rot="R90" display="off"/>
 </element>
 </elements>
@@
 <contactref element="U3" pad="2"/>
 <contactref element="U1" pad="GND"/>
-<wire x1="-5.66" y1="-11.91" x2="0.22" y2="-17.8451" width="0" layer="19" extent="1-1"/>
-<wire x1="4.6" y1="-5.4" x2="-5.66" y2="-11.91" width="0" layer="19" extent="1-1"/>
+<contactref element="U2" pad="17" route="any" routetag="G$1.GND"/>
+<contactref element="U2" pad="1" route="any" routetag="G$1.GND"/>
+<contactref element="U2" pad="37" route="any" routetag="G$1.GND"/>
+<contactref element="U2" pad="40" route="any" routetag="G$1.GND"/>
+<contactref element="U2" pad="38" route="any" routetag="G$1.GND"/>
+<contactref element="U2" pad="44" route="any" routetag="G$1.GND"/>
+<contactref element="U2" pad="8" route="any" routetag="G$1.GND"/>
+<contactref element="U2" pad="41" route="any" routetag="G$1.GND"/>
+<contactref element="U2" pad="12" route="any" routetag="G$1.GND"/>
+<contactref element="U2" pad="39" route="any" routetag="G$1.GND"/>
+<contactref element="U2" pad="49" route="any" routetag="G$1.GND"/>
+<contactref element="U2" pad="10" route="any" routetag="G$1.GND"/>
+<contactref element="U2" pad="3" route="any" routetag="G$1.GND"/>
+<contactref element="U2" pad="23" route="any" routetag="G$1.GND"/>
+<contactref element="U2" pad="7" route="any" routetag="G$1.GND"/>
+<contactref element="U2" pad="9" route="any" routetag="G$1.GND"/>
+<contactref element="U2" pad="11" route="any" routetag="G$1.GND"/>
+<contactref element="U2" pad="5" route="any" routetag="G$1.GND"/>
+<wire x1="4.37" y1="6" x2="-7.636" y2="4.044" width="0" layer="19" extent="1-1"/>
+<wire x1="0.22" y1="-17.8451" x2="4.37" y2="6" width="0" layer="19" extent="1-1"/>
+<wire x1="4.6" y1="-5.4" x2="4.37" y2="6" width="0" layer="19" extent="1-1"/>
 <wire x1="0.3102" y1="9.353" x2="4.6" y2="-5.4" width="0" layer="19" extent="1-1"/>
 <wire x1="4.8502" y1="13.413" x2="4.1002" y2="13.443" width="0" layer="19" extent="1-1"/>
@@
 <contactref element="U1" pad="PAD"/>
 </signal>
+<signal name="VCC">
+<contactref element="U2" pad="24"/>
+<contactref element="U2" pad="25"/>
+<wire x1="-11.636" y1="0.044" x2="-11.136" y2="0.044" width="0" layer="19" extent="1-1"/>
+</signal>
+<signal name="V_CORE">
+<contactref element="U2" pad="27"/>
+</signal>
+<signal name="V_DCDC_OUT">
+<contactref element="U2" pad="26"/>
+</signal>
+<signal name="V_BCKP">
+<contactref element="U2" pad="16"/>
+</signal>
 </signals>

Commit message: moar edits
revision 3 to main board layout, inclusion of TPL5110, possible future exchange for RV-3028
Parts:
- added C3, C4: 10 uF, rcl:C0201
- added C5: 4.7uF, SparkFun-Capacitors:0603
- added C6: 0.1uF, SparkFun-Capacitors:0603
- added C7: 10uF, SparkFun-Capacitors:0603
- added C8: 1.0uF, SparkFun-Capacitors:0402
- added D1: 1A/23V/620mV, SparkFun-DiscreteSemi:SOD-323
- added J4: (no value), SparkFun-Connectors:1X04_1.27MM_NO_SILK
- added J5: (no value), SparkFun-Connectors:USB-MICROB-PTH-MILL
- added L2: 2.2uH, SparkFun-Coils:0806
- added Q2: 3.1A/30V/105mΩ, SparkFun-DiscreteSemi:SOT23-3
- added R4: 10k, SparkFun-Resistors:0402
- added R5: 10k, rcl:R0201
- added U5: 3.3V, SparkFun-IC-Power:SOT23-5
- added Y1: 32.768kHz, SparkFun-Clocks:CRYSTAL-SMD-3.2X1.5MM
- added Y2: W3011, SparkFun-GPS:W3011
- U2: value UBLOX_ZOE_M8Q-0-10 -> UBLOX_ZOE_M8-0-10
- moved U2 30.6 mm to (17.7, -11.7)
- moved U4 18.8 mm to (16.6, 8.63)
Connections:
- removed net GNDANA: U1.GNDANA
- removed net PAD: U1.PAD
- removed net VCC: U2.24, U2.25
- removed net VDDANA: U1.VDD
- removed net VDDCORE: U1.VDDCORE
- removed net VDDIN: U1.VDDIN
- removed net V_BCKP: U2.16
- removed net V_CORE: U2.27
- removed net V_DCDC_OUT: U2.26
- new net !INT: U2.43
- new net !RESET: J4.1, U2.20
- new net !SAFEBOOT: U2.34
- new net 3.3V: C3.1, C6.1, C7.1, C8.1, R5.2, U1.VDD, U1.VDDIN, U2.24, U2.25, U4.3.3V, U5.5
- new net ANT: U2.4
- new net D+: J5.D+, U1.PA25
- new net D-: J5.D-, U1.PA24
- new net D13: U1.PA10
- new net D7: U1.PA04
- new net DAC: U1.PA02
- new net D_SEL: U2.48
- new net FLASH_CS: U1.PA19
- new net FLASH_MISO: U1.PA18
- new net FLASH_MOSI: U1.PA16
- new net FLASH_SCK: U1.PA17
- new net MISO: U1.PA05, U4.MISO
- new net MOSI: U1.PA06, U4.MOSI
- new net N$10: C4.1, U1.VDDCORE
- new net N$13: C5.1, L2.1, U2.27
- new net N$14: U2.18, Y1.P$2
- new net N$15: U2.19, Y1.P$1
- new net N$4: L2.2, U2.26
- new net RESET: U1.RES
- new net RFM_ANT: U4.ANT
- new net RFM_CS: R5.1, U1.PA00, U4.NSS
- new net RFM_INT: U1.PA01, U4.DIO0
- new net RFM_RST: U1.PA22, U4.!RESET
- new net RX: U1.PA23
- new net RXI/MOSI: U2.22
- new net SCK: U1.PA07, U4.SCK
- new net SCL: U1.PA09, U2.32
- new net SDA: U1.PA08, U2.2
- new net SWCLK: J4.3, U1.PA30
- new net SWDIO: J4.4, U1.PA31
- new net TIMEPULSE: U2.33
- new net TXO/MISO: U2.21
- new net V_BATT: Q2.3, U2.16
- new net V_USB: D1.A, J5.VBUS, Q2.1, R4.2
- net GND: now also C3.2, C4.2, C5.2, C6.2, C7.2, C8.2, J4.2, J5.GND, J5.SHIELD, J5.SHIELD10, J5.SHIELD2, J5.SHIELD3, J5.SHIELD4, J5.SHIELD5, J5.SHIELD6, J5.SHIELD7, J5.SHIELD8, J5.SHIELD9, R4.1, U1.GNDANA, U1.PAD, U2.29, U2.31, U2.46, U2.47, U4.GND@1, U4.GND@2, U4.GND@3, U5.2
- net VIN: now also D1.C, Q2.2, U5.1, U5.3
Other:
- board size 24.6 x 16.5 mm -> 24.8 x 17.2 mm
