File: EAGLE/GPS_radiologger_v4.brd (EAGLE design)
At the start: 24.8 x 17.2 mm, 39 parts, among them Q1 1.1A/60V/600mΩ, Q2 3.1A/30V/105mΩ, U1 ATSAMD21E18A-U, U2 UBLOX_ZOE_M8-0-10, U3 TPL5110, U4 RFM95W, U5 3.3V, Y1 32.768kHz, Y2 GPS_CHIP_ANTENNAW3011

Commit message: moar edits
revision 3 to main board layout, inclusion of TPL5110, possible future exchange for RV-3028
Parts:
- removed C8: 1.0uF, SparkFun-Capacitors:0402
- removed JP1, JP2, JP3, JP4, JP5, JP6: (no value), pinhead:1X01
- removed L1: 22 uH, LPS4012-103MRB:IND_LPS4012-103MRB
- removed R4: 10k, SparkFun-Resistors:0402
- removed RPG1, RPG2, RSD2, RTERM2: (no value), resistor:R0201
- removed RSD1, RTERM1: (no value), rcl:R0402
- added FB1: FERRITE_BEAD-120_OHM-0402, SparkFun-Coils:0402
- added J1: (no value), SparkFun-Connectors:1X01_OFFSET
- added J2: (no value), SparkFun-Connectors:1X02
- added R5: 10k, rcl:R0201
- C1: value 4.7uF -> 47 pF; device resistor:C0402 -> rcl:C0201
- C2: value 10uF -> 10 uF; device resistor:C0402 -> rcl:C0201
- C5: value 4.7uF -> 4.7 uF; device SparkFun-Capacitors:0603 -> rcl:C0201
- C6: value 0.1uF -> 0.1 uF; device SparkFun-Capacitors:0603 -> rcl:C0201
- C7: value 10uF -> 1 uF; device SparkFun-Capacitors:0603 -> rcl:C0201
- R1: value 6.34M -> 10; device resistor:R0201 -> rcl:R0201
- R2: value 14.7M -> 30 k; device resistor:R0201 -> rcl:R0603
- R3: value 20k -> 10k; device resistor:R0201 -> rcl:R0201
- U$2: value ADP5090 -> MB85RC64TA; device ADP5090_LFCSP-16-3X3:LFCSP-16-3X3 -> Fujitsu_FRAM:8-SON_2X3
- Y2: value GPS_CHIP_ANTENNAW3011 -> W3011
- moved U4 98.2 mm to (18.1, 9.24), turned to 90 degrees
- moved C6 80.0 mm to (16.6, -1.94)
- moved C5 68.5 mm to (2.06, -3.74)
- moved Y1 61.0 mm to (-11.2, -10.9), turned to 180 degrees
- moved L2 59.3 mm to (-7.02, -12.9), turned to 90 degrees
- moved J5 53.4 mm to (38.0, 8.52), turned to 270 degrees
- moved J4 48.8 mm to (37.0, 14.8)
- moved C7 47.8 mm to (7.73, -6.95)
- moved D1 46.4 mm to (23.8, -15.4)
- moved R2 44.9 mm to (20.2, -28.8), turned to 180 degrees
- moved Q2 41.2 mm to (-9.48, -1.47)
- moved U5 38.3 mm to (-0.08, -17.9), turned to 180 degrees
- moved R3 31.9 mm to (29.1, -3.63)
- moved U2 28.6 mm to (-10.6, -15.3), turned to 180 degrees
- moved C3 24.4 mm to (17.1, -27.4)
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Connections:
- removed net BAT: JP4.1, U$2.10
- removed net D5: U1.PA00
- removed net D6: U1.PA01
- removed net D7: U1.PA04
- removed net DIS_SW: JP3.1, U$2.14
- removed net N$1: R1.1, R2.2, U$2.5
- removed net N$11: RPG1.2, RSD1.2, RTERM1.2, U$2.15
- removed net N$2: C2.1, U$2.6
- removed net N$5: R3.2, U$2.4
- removed net N$6: U3.1, U3.6
- removed net N$7: RTERM1.1, RTERM2.2, U$2.2
- removed net N$8: RPG1.1, RPG2.2, U$2.16
- removed net PGOOD: JP1.1, U$2.13
- removed net RX: U1.PA23
- removed net SYS: JP2.1, U$2.11
- removed net TX: U1.PA22
- removed net VDD_OUT: Q1.3
- new net RFM_ANT: J1.1, U4.ANT
- new net RFM_CS: R5.1, U1.PA00, U4.NSS
- new net RFM_INT: U1.PA01, U4.DIO0
- new net RFM_RST: U1.PA04, U4.!RESET
- net 3.3V: now also Q1.3, R1.2, R5.2, U$2.P$5, U4.3.3V; no longer C7.1, C8.1, U5.5
- net ANT: now also FB1.1, Y2.1
- net DELAY/M_DRIVE: now also R2.1
- net DONE: now also U1.PA22
- net GND: now also R2.2, U$2.P$1, U$2.P$2, U$2.P$3, U$2.P$4, U$2.P$9, U4.GND@1, U4.GND@2, U4.GND@3, Y2.2, Y2.3; no longer C8.2, JP5.1, R2.1, R4.1, RPG2.1, RSD2.1, RTERM2.1, U$2.3, U$2.8, U$2.EXP
- net MISO: now also U4.MISO
- net MOSI: now also U4.MOSI
- net N$3: now also U$2.P$6; no longer L1.2, U$2.9
- net N$9: now also C1.1, FB1.2, R1.1; no longer RSD1.1, RSD2.2, U$2.1
- net SCK: now also U4.SCK
- net SCL: now also U$2.P$7
- net SDA: now also U$2.P$8
- net VDD: now also C2.1, C7.1, U3.1, U3.6, U5.5
- net VIN: no longer C1.1, JP6.1, L1.1, R1.2, U$2.7
- net V_BATT: now also J2.2
- net V_USB: now also J2.1, R3.2; no longer R4.2
Routing:
- net VIN: track 23.7 -> 0.00 mm
- net GND: track 25.4 -> 4.96 mm, vias 1 -> 0
- net N$8: track 4.32 -> 0.00 mm
- net N$11: track 4.19 -> 0.00 mm
- net N$3: track 3.53 -> 0.00 mm
- net N$2: track 3.19 -> 0.00 mm
- net N$9: track 3.19 -> 0.00 mm
- net DIS_SW: track 3.03 -> 0.00 mm
- net N$1: track 2.55 -> 0.00 mm
- net PGOOD: track 2.12 -> 0.00 mm
- net BAT: track 1.65 -> 0.00 mm
- net SYS: track 1.58 -> 0.00 mm
- net N$7: track 1.35 -> 0.00 mm
- net N$5: track 1.10 -> 0.00 mm
Other:
- board size 24.8 x 17.2 mm -> 28.6 x 18.7 mm
