File: EAGLE/GPS_radiologger_v14.brd (EAGLE design)
At the start: 36 x 23 mm, 38 parts, among them IC4 CAT24M01HU5I-GT3, U1 TYPEABZ, U2 UBLOX_ZOE_M8-0-10, U3 MICROCHIP_MCP1810T-33I-J8AMIC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, U5 BME680BME680, Y1 32.768kHz, Y2 W3011

Commit message: rolling along with v14 / implementation of solar power
Parts:
- added U4: SPV1050, STM-SPV1050_V2:SPV1050
Connections:
- new net IN_HV: U4.P$20
- new net IN_LV: U4.P$16
- new net L_HV: U4.P$19
Changed lines of the file:
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@@
 <layer number="154" name="FabDoc2" color="7" fill="1" visible="no" active="no"/>
 <layer number="155" name="FabDoc3" color="7" fill="1" visible="no" active="no"/>
+<layer number="160" name="FAB" color="7" fill="1" visible="no" active="yes"/>
+<layer number="166" name="AntennaArea" color="7" fill="1" visible="yes" active="yes"/>
+<layer number="168" name="4mmHeightArea" color="7" fill="1" visible="yes" active="yes"/>
 <layer number="191" name="mNets" color="7" fill="1" visible="no" active="no"/>
 <layer number="192" name="mBusses" color="7" fill="1" visible="no" active="no"/>
@@
 <layer number="250" name="Descript" color="3" fill="1" visible="no" active="no"/>
 <layer number="251" name="SMDround" color="12" fill="11" visible="no" active="no"/>
+<layer number="252" name="RM45" color="7" fill="1" visible="no" active="yes"/>
 <layer number="253" name="Extra" color="7" fill="1" visible="yes" active="yes"/>
 <layer number="254" name="cooling" color="7" fill="1" visible="no" active="no"/>
@@
 <attribute name="VALUE" x="21.5" y="-2.739" size="0.6096" layer="27" font="vector" ratio="20" align="top-center"/>
 </element>
+<element name="U4" library="STM-SPV1050_V2" package="SPV1050" value="SPV1050" x="2.65" y="-7.4" smashed="yes">
+<attribute name="NAME" x="-0.35" y="-5.4" size="1.27" layer="25"/>
+<attribute name="VALUE" x="-0.75" y="-10.8" size="1.27" layer="27"/>
+</element>
 </elements>
 <signals>
@@
 <wire x1="22.4" y1="-1.85" x2="19.34661875" y2="8.750540625" width="0" layer="19" extent="1-1"/>
 </signal>
+<signal name="IN_LV">
+<contactref element="U4" pad="P$16"/>
+</signal>
+<signal name="IN_HV">
+<contactref element="U4" pad="P$20"/>
+</signal>
+<signal name="L_HV">
+<contactref element="U4" pad="P$19"/>
+</signal>
 </signals>
