File: EAGLE/v_14/CMWX_LoRa_GPS_v14.brd (EAGLE design)
At the start: 36 x 23 mm, 39 parts, among them IC4 CAT24M01HU5I-GT3, U1 TYPEABZ, U2 UBLOX_ZOE_M8-0-10, U3 MICROCHIP_MCP1810T-33I-J8AMIC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, U4 SPV1050, U5 BME680BME680, Y1 32.768kHz, Y2 W3011

Commit message: rolling along with v14 / implementation of solar power
Parts:
- removed J2: (no value), SparkFun-Connectors:1X01_SMALL
- added C13: 47uF, rcl:C0201
- added C14: 4.7 uF, rcl:C0201
- added C4: 10nF, rcl:C0201
- added JP2: JUMPER-SMT_2_NC_TRACE_NO-SILK, SparkFun-Jumpers:SMT-JUMPER_2_NC_TRACE_NO-SILK
- added R10: 6.2M, rcl:R0201
- added R11: 1M, rcl:R0201
- added R12, R8: 3M, rcl:R0201
- added R9: 9.1M, rcl:R0201
- added U$1: LPS3015, coilcraft_custom:LPS_3015
- added U$2: NITINOL_ANTENNA, Antenna_mounts:ICARUS_NITINOL_ANTENNA
- added U$3: ICARUS_FULL, TrisolX_Solar_Cells:ICARUS_FULL
- moved U4 22.6 mm to (3.40, 15.2)
- moved C3 20.3 mm to (-1.10, 18.4)
- moved L1 18.1 mm to (13.4, 14.3), turned to 90 degrees
- moved U5 16.8 mm to (32.5, 18.7)
- moved C6 9.55 mm to (11.3, 16.1)
- moved Y1 9.55 mm to (8.67, 16.5)
- moved C5 9.55 mm to (11.3, 16.7)
- moved U2 9.55 mm to (10.1, 13.4)
- moved R5 7.89 mm to (6.45, 15.7), turned to 0 degrees
- moved R4 7.88 mm to (6.45, 13.6), turned to 0 degrees
- moved PDTA143TMB,1 7.33 mm to (6.45, 16.7), turned to 90 degrees
- moved PDTA143TMB,315 7.31 mm to (6.45, 14.6), turned to 90 degrees
- moved JP1 7.07 mm to (6.65, 11.8)
- moved C1 4.72 mm to (29.4, 16.8)
- moved C10 4.72 mm to (15.6, 16.4)
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Connections:
- removed net IN_HV: U4.P$20
- removed net IN_LV: U4.P$16
- removed net L_HV: U4.P$19
- new net N$10: JP2.1, U4.P$14
- new net N$11: C14.1, R8.2, U$1.P$1, U$3.P$1, U4.P$1, U4.P$13
- new net N$12: C13.1, R10.2, U4.P$15
- new net N$13: C4.1, U4.P$3
- new net N$4: U$1.P$2, U4.P$16
- new net N$6: R8.1, R9.2, U4.P$2
- new net N$8: R10.1, R11.2, U4.P$10
- new net N$9: R11.1, R12.2, U4.P$9
- net ANT: now also U$2.P$1, U$2.P$2, U$2.P$3, U$2.P$4; no longer J2.P$1
- net BAT: now also JP2.2
- net GND: now also C13.2, C14.2, C4.2, R12.1, R9.1, U$3.P$2, U4.P$18, U4.P$19, U4.P$20, U4.P$21, U4.P$4, U4.P$5, U4.P$6
Routing:
- net SDA: track 78.1 -> 0.00 mm, vias 4 -> 0
- net SCL: track 75.6 -> 0.00 mm, vias 3 -> 0
- net BAT: track 43.1 -> 0.00 mm, vias 2 -> 0
- net SCD_PWR: track 36.3 -> 0.00 mm, vias 1 -> 0
- net GND: track 31.8 -> 0.00 mm, vias 81 -> 0
- net POWER: track 22.2 -> 0.00 mm, vias 7 -> 0
- net SCD_PDTA: track 20.7 -> 0.00 mm, vias 2 -> 0
- net ZOE_PDTA: track 19.8 -> 0.00 mm, vias 2 -> 0
- net VBUS: track 16.9 -> 0.00 mm, vias 1 -> 0
- net ZOE_PWR: track 7.67 -> 0.00 mm
- net RST: track 7.03 -> 0.00 mm
- net DM: track 5.02 -> 0.00 mm, vias 1 -> 0
- net GPS_ANT: track 4.28 -> 0.00 mm
- net ANT: track 3.71 -> 0.00 mm
- net N$1: track 3.28 -> 0.00 mm
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Other:
- board size 36 x 23 mm -> 36 x 21.6 mm
