File: EAGLE/v_14/GPS_radiologger_v14.brd (EAGLE design)
At the start: 36 x 23 mm, 39 parts, among them IC4 CAT24M01HU5I-GT3, U1 TYPEABZ, U2 UBLOX_ZOE_M8-0-10, U3 MICROCHIP_MCP1810T-33I-J8AMIC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, U4 SPV1050, U5 BME680BME680, Y1 32.768kHz, Y2 W3011

Commit message: rolling along with v14 / implementation of solar power
Connections:
- net GND: now also U4.P$18, U4.P$21, U4.P$4
