File: EAGLE/v_14/GPS_radiologger_v14.sch (EAGLE design)
At the start: 39 parts, among them IC4 CAT24M01HU5I-GT3, U1 TYPEABZ, U2 UBLOX_ZOE_M8-0-10, U3 MICROCHIP_MCP1810T-33I-J8AMIC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, U4 SPV1050, U5 BME680BME680, Y1 32.768kHz, Y2 W3011

Commit message: rolling along with v14 / implementation of solar power
Connections:
- net GND: now also U4.GND, U4.PAD, U4.PGND
Other:
- moved on the sheet: C12, C3, C8, J7, PDTA143TMB,1, PDTA143TMB,315, R4, R5, U3, U5, Y2
