File: EAGLE/v_14/CMWX_LoRa_GPS_v14.sch (EAGLE design)
At the start: 39 parts, among them IC4 CAT24M01HU5I-GT3, U1 TYPEABZ, U2 UBLOX_ZOE_M8-0-10, U3 MICROCHIP_MCP1810T-33I-J8AMIC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, U4 SPV1050, U5 BME680BME680, Y1 32.768kHz, Y2 W3011

Commit message: rolling along with v14 / implementation of solar power
Parts:
- removed J2: (no value), SparkFun-Connectors:CONN_01PTH_NO_SILK_SMALL
- added C13: 47uF, rcl:C-EUC0201
- added C14: 4.7 uF, rcl:C-EUC0201
- added C4: 10nF, rcl:C-EUC0201
- added JP2: JUMPER-SMT_2_NC_TRACE_NO-SILK, SparkFun-Jumpers:JUMPER-SMT_2_NC_TRACE_NO-SILK
- added R10: 6.2M, rcl:R-EU_R0201
- added R11: 1M, rcl:R-EU_R0201
- added R12, R8: 3M, rcl:R-EU_R0201
- added R9: 9.1M, rcl:R-EU_R0201
- added U$1: LPS3015, coilcraft_custom:LPS3015
- added U$2: NITINOL_ANTENNA, Antenna_mounts:NITINOL_ANTENNA
- added U$3: ICARUS_FULL, TrisolX_Solar_Cells:ICARUS_FULL
Connections:
- new net N$10: JP2.1, U4.BATT
- new net N$11: C14.1, R8.2, U$1.1, U$3.PLUS, U4.CONF, U4.MPP
- new net N$12: C13.1, R10.2, U4.STORE
- new net N$13: C4.1, U4.MPP_REF
- new net N$4: U$1.2, U4.IN_LV
- new net N$6: R8.1, R9.2, U4.MPP_SET
- new net N$8: R10.1, R11.2, U4.UVP
- new net N$9: R11.1, R12.2, U4.EOC
- net ANT: now also U$2.SIGNAL; no longer J2.1
- net BAT: now also JP2.2
- net GND: now also C13.2, C14.2, C4.2, R12.1, R9.1, U$3.MINUS, U4.GND, U4.IN_HV, U4.LDO1_EN, U4.LDO2_EN, U4.L_HV, U4.PAD, U4.PGND
Other:
- note added: "1/4 lambda = 86.3 mm at 868 MHz"
- note added: "CO2 Concentration Sensor Sensirion SCD30"
- note added: "Cut JP2 for battery only operation"
- note added: "Default Address 0x61"
- note added: "General VOC/ RH/ Temp Bosch BME680"
- note added: "Include castellated holes for edge connection"
- note added: "Power Storage - LiPo"
- note added: "future - implement the SGX MICS-2714 Sensor for VOC/NOx"
- note added: "rev14 - add SPV1050 and associated passives"
- note added: "rev14 - add solar cell"
- note added: "rev14 - castellated vias for all programming pins"
- note added: "rev14 - include new antenna land"
- note added: "v14"
- note removed: "Power Supply - Lithium Polymer"
- note removed: "SCD30 Breakout Pins"
- note removed: "v12"
- moved on the sheet: C12, C3, C8, IC4, J1, J3, J4, J5, J6, J7, PDTA143TMB,1, PDTA143TMB,315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

Commit message: latest edits v14
Parts:
- removed J4: (no value), SparkFun-Connectors:CONN_031X03_1.27_NO_SILK
- removed J5, J6: (no value), SparkFun-Connectors:CONN_041.27MM_NO_SILK
- added U$4: ICARUS_FULL, TrisolX_Solar_Cells:ICARUS_FULL
- added U$5: ALBERT_ZIGZAG-ISP, Zigzag ISP connector:ALBERT_ZIGZAG-ISP
- C11: value 0.1 uF -> 0.1uF; device rcl:C-EUC0201 -> SparkFun-Capacitors:0.1UF-0402T-16V-10%
- C13: value 47uF -> 100 uF
- U$2: value NITINOL_ANTENNA -> NITINOL_ANTENNA_SHORT; device Antenna_mounts:NITINOL_ANTENNA -> Antenna_mounts:NITINOL_ANTENNA_SHORT
Connections:
- net BOOT: now also U$5.BOOT; no longer J5.1
- net DM: no longer J6.2
- net DP: no longer J6.3
- net GND: now also U$5.GND; no longer J6.4
- net POWER: now also U$5.POWER; no longer C6.1, J4.1, U2.VCC
- net RST: now also U$5.RESET; no longer J5.4
- net RX: no longer J4.2
- net SWDCLK: now also U$5.SWDCLK; no longer J5.2
- net SWDIO: now also U$5.SWDIO; no longer J5.3
- net TX: no longer J4.3
- net VBUS: no longer J6.1
- net ZOE_PWR: now also C6.1, U2.VCC
Other:
- note added: "rev14 - add in zigzag connector for SWD programming"
- note removed: "rev14 - add POWER pin for SWD"
- note removed: "rev14 - castellated vias for all programming pins"
- moved on the sheet: C12, C13, C14, C4, C8, JP2, PDTA143TMB,315, R10, R11, R12, R4, R8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
