File: EAGLE/v_14/CMWX_LoRa_GPS_v14_CAM.brd (EAGLE design)
At the start: 38.6 x 23 mm, 49 parts, among them IC4 CAT24M01HU5I-GT3, U1 TYPEABZ, U2 UBLOX_ZOE_M8-0-10, U3 MICROCHIP_MCP1810T-33I-J8AMIC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, U4 SPV1050, U5 BME680BME680, Y1 32.768kHz, Y2 W3011

Commit message: latest edits v14
Parts:
- removed U$5: ALBERT_ZIGZAG-ISP, Zigzag ISP connector:ALBERT_ZIGZAG-ISP
- added J4: (no value), SparkFun-Connectors:1X03_1.27MM_NO_SILK
- added J5, J6: (no value), SparkFun-Connectors:1X04_1.27MM_NO_SILK
- C11: value 0.1uF -> 0.1 uF; device SparkFun-Capacitors:0402-TIGHT -> rcl:C0201
- C13: value 100 uF -> 47uF
- U$2: value NITINOL_ANTENNA_SHORT -> NITINOL_ANTENNA; device Antenna_mounts:ICARUS_NITINOL_ANTENNA_SHORT -> Antenna_mounts:ICARUS_NITINOL_ANTENNA
- moved C14 44.1 mm to (-9.55, -43.5), turned to 0 degrees
- moved JP2 39.1 mm to (-3.05, -37.6)
- moved C13 36.6 mm to (-0.10, -38.5), turned to 0 degrees
- moved C4 30.9 mm to (-0.10, -35.0), turned to 0 degrees
- moved R12 26.9 mm to (-0.10, -31.6)
- moved R11 24.1 mm to (-0.10, -28.1)
- moved R10 21.7 mm to (-0.10, -24.6)
- moved U4 21.3 mm to (3.40, 15.2)
- moved R9 18.8 mm to (-0.10, -21.1)
- moved R4 18.7 mm to (6.45, 13.6), turned to 0 degrees
- moved PDTA143TMB,315 18.2 mm to (6.45, 14.6), turned to 90 degrees
- moved R5 17.8 mm to (6.45, 15.7), turned to 0 degrees
- moved U5 17.7 mm to (32.5, 18.7), turned to 180 degrees
- moved PDTA143TMB,1 17.5 mm to (6.45, 16.7), turned to 90 degrees
- moved R8 16.2 mm to (-0.10, -17.6)
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Connections:
- net ANT: now also U$2.P$1, U$2.P$2, U$2.P$3, U$2.P$4; no longer U$2.1, U$2.2, U$2.3
- net BOOT: now also J5.1; no longer U$5.4
- net DM: now also J6.2
- net DP: now also J6.3
- net GND: now also J6.4; no longer U$5.5
- net POWER: now also C6.1, J4.1, U2.24, U2.25; no longer U$5.6
- net RST: now also J5.4; no longer U$5.1
- net RX: now also J4.2
- net SWDCLK: now also J5.2; no longer U$5.3
- net SWDIO: now also J5.3; no longer U$5.2
- net TX: now also J4.3
- net VBUS: now also J6.1
- net ZOE_PWR: no longer C6.1, U2.24, U2.25
Routing:
- net GND: track 2.72 -> 0.00 mm
- net N$8: track 1.39 -> 0.00 mm
- net N$9: track 1.29 -> 0.00 mm
- net N$12: track 0.65 -> 0.00 mm
Other:
- board size 38.6 x 23 mm -> 36 x 21.6 mm
