File: EAGLE/v_14/CMWX_LoRa_GPS_v14_CAM.sch (EAGLE design)
At the start: 49 parts, among them IC4 CAT24M01HU5I-GT3, U1 TYPEABZ, U2 UBLOX_ZOE_M8-0-10, U3 MICROCHIP_MCP1810T-33I-J8AMIC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, U4 SPV1050, U5 BME680BME680, Y1 32.768kHz, Y2 W3011

Commit message: latest edits v14
Parts:
- removed U$5: ALBERT_ZIGZAG-ISP, Zigzag ISP connector:ALBERT_ZIGZAG-ISP
- added J4: (no value), SparkFun-Connectors:CONN_031X03_1.27_NO_SILK
- added J5, J6: (no value), SparkFun-Connectors:CONN_041.27MM_NO_SILK
- C11: value 0.1uF -> 0.1 uF; device SparkFun-Capacitors:0.1UF-0402T-16V-10% -> rcl:C-EUC0201
- U$2: value NITINOL_ANTENNA_SHORT -> NITINOL_ANTENNA; device Antenna_mounts:NITINOL_ANTENNA_SHORT -> Antenna_mounts:NITINOL_ANTENNA
Connections:
- net BOOT: now also J5.1; no longer U$5.BOOT
- net DM: now also J6.2
- net DP: now also J6.3
- net GND: now also J6.4; no longer U$5.GND
- net POWER: now also C6.1, J4.1, U2.VCC; no longer U$5.POWER
- net RST: now also J5.4; no longer U$5.RESET
- net RX: now also J4.2
- net SWDCLK: now also J5.2; no longer U$5.SWDCLK
- net SWDIO: now also J5.3; no longer U$5.SWDIO
- net TX: now also J4.3
- net VBUS: now also J6.1
- net ZOE_PWR: no longer C6.1, U2.VCC
Other:
- note added: "rev14 - add POWER pin for SWD"
- note added: "rev14 - castellated vias for all programming pins"
- note removed: "rev14 - add in zigzag connector for SWD programming"
