File: EAGLE/v15/GPS_radiologger_v15.brd (EAGLE design)
At the start: 38.6 x 23 mm, 48 parts, among them IC4 CAT24M01HU5I-GT3, U1 TYPEABZ, U2 UBLOX_ZOE_M8-0-10, U3 MICROCHIP_MCP1810T-33I-J8AMIC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, U4 SPV1050, U5 BME680BME680, Y1 32.768kHz, Y2 W3011

Commit message: recent general edits
Parts:
- removed C2: 10 uF, rcl:C0201
- removed JP2: JUMPER-SMT_2_NC_TRACE_NO-SILK, SparkFun-Jumpers:SMT-JUMPER_2_NC_TRACE_NO-SILK
- added J2: (no value), SparkFun-Connectors:1X02_NO_SILK
- moved C13 10.7 mm to (17.0, 14.6), turned to 0 degrees
- moved C10 2.60 mm to (19.5, 14.2)
- moved C9 2.60 mm to (19.0, 14.2)
- moved C12 2.55 mm to (19.4, 16.7)
- moved Y1 2.55 mm to (14.3, 15.6)
- moved U3 2.55 mm to (17.5, 16.6)
- moved C1 2.55 mm to (30.8, 17.9)
- moved C14 2.55 mm to (19.4, 9.75)
- moved C4 2.55 mm to (19.4, 11.7)
- moved C6 2.55 mm to (13.9, 13.7)
- moved C7 2.55 mm to (14.2, 16.8)
- moved C8 2.55 mm to (15.4, 16.1)
- moved IC4 2.55 mm to (11.1, 11.2)
- moved PDTA143TMB,1 2.55 mm to (13.8, 7.93)
- moved PDTA143TMB,315 2.55 mm to (13.8, 9.08)
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Connections:
- removed net N$10: JP2.1, U4.P$14
- net BAT: now also U4.P$14; no longer JP2.2
- net GND: no longer C2.1
- net POWER: no longer C2.2
- net RX: now also J2.1
- net TX: now also J2.2
Routing:
- net RX: track 0.00 -> 23.3 mm, vias 0 -> 1
- net TX: track 0.00 -> 21.1 mm, vias 0 -> 1
- net BAT: track 17.6 -> 24.6 mm
- net N$10: track 3.58 -> 0.00 mm
- net SCD_PWR: track 21.9 -> 24.5 mm
- net GPS_ANT: track 4.66 -> 7.21 mm
- net N$11: track 7.65 -> 5.48 mm
- net GND: track 76.5 -> 78.4 mm, vias 67 -> 92
- net RST: track 8.64 -> 10.6 mm
- net POWER: track 67.7 -> 66.0 mm
- net SCL: track 61.6 -> 63.2 mm
- net N$12: track 8.54 -> 6.98 mm
- net SDA: track 50.0 -> 51.5 mm
- net VOLT_MEAS: track 33.9 -> 34.4 mm
Other:
- outline, holes or cut-outs redrawn
- board text added: "+"
- board text added: "-"
- board text added: "Pollution Tag v1.15.0"
