File: EAGLE/v15/GPS_radiologger_v15.sch (EAGLE design)
At the start: 48 parts, among them IC4 CAT24M01HU5I-GT3, U1 TYPEABZ, U2 UBLOX_ZOE_M8-0-10, U3 MICROCHIP_MCP1810T-33I-J8AMIC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, U4 SPV1050, U5 BME680BME680, Y1 32.768kHz, Y2 W3011

Commit message: recent general edits
Parts:
- removed C2: 10 uF, rcl:C-EUC0201
- removed JP2: JUMPER-SMT_2_NC_TRACE_NO-SILK, SparkFun-Jumpers:JUMPER-SMT_2_NC_TRACE_NO-SILK
- added J2: (no value), SparkFun-Connectors:CONN_021X02_NO_SILK
- C13: value 100 uF -> 47 uF
Connections:
- removed net N$10: JP2.1, U4.BATT
- net BAT: now also U4.BATT; no longer JP2.2
- net GND: no longer C2.1
- net POWER: no longer C2.2
- net RX: now also J2.1
- net TX: now also J2.2
Changed lines of the file:
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@@
 <setting verticaltext="up"/>
 </settings>
-<grid distance="0.1" unitdist="inch" unit="inch" style="lines" multiple="1" display="no" altdistance="0.01" altunitdist="inch" altunit="inch"/>
+<grid distance="0.05" unitdist="inch" unit="inch" style="lines" multiple="1" display="no" altdistance="0.01" altunitdist="inch" altunit="inch"/>
 <layers>
 <layer number="1" name="Top" color="4" fill="1" visible="no" active="no"/>
@@
 <part name="C5" library="rcl" library_urn="urn:adsk.eagle:library:334" deviceset="C-EU" device="C0201" package3d_urn="urn:adsk.eagle:package:23690/2" value="4.7 uF"/>
 <part name="C6" library="rcl" library_urn="urn:adsk.eagle:library:334" deviceset="C-EU" device="C0201" package3d_urn="urn:adsk.eagle:package:23690/2" value="0.1 uF"/>
-<part name="C2" library="rcl" library_urn="urn:adsk.eagle:library:334" deviceset="C-EU" device="C0201" package3d_urn="urn:adsk.eagle:package:23690/2" value="10 uF"/>
 <part name="C9" library="rcl" library_urn="urn:adsk.eagle:library:334" deviceset="C-EU" device="C0201" package3d_urn="urn:adsk.eagle:package:23690/2" value="1 uF"/>
 <part name="U1" library="Kris" deviceset="TYPEABZ" device=""/>
@@
 <part name="R12" library="rcl" library_urn="urn:adsk.eagle:library:334" deviceset="R-EU_" device="R0201" package3d_urn="urn:adsk.eagle:package:26117/2" value="3M"/>
 <part name="C4" library="rcl" library_urn="urn:adsk.eagle:library:334" deviceset="C-EU" device="C0201" package3d_urn="urn:adsk.eagle:package:23690/2" value="10nF"/>
-<part name="C13" library="rcl" library_urn="urn:adsk.eagle:library:334" deviceset="C-EU" device="C0805K" package3d_urn="urn:adsk.eagle:package:23681/2" value="100 uF"/>
-<part name="JP2" library="SparkFun-Jumpers" deviceset="JUMPER-SMT_2_NC_TRACE" device="_NO-SILK" package3d_urn="urn:adsk.eagle:package:39286/1"/>
+<part name="C13" library="rcl" library_urn="urn:adsk.eagle:library:334" deviceset="C-EU" device="C0805K" package3d_urn="urn:adsk.eagle:package:23681/2" value="47 uF"/>
 <part name="U$2" library="Antenna_mounts" deviceset="NITINOL_ANTENNA_SHORT" device=""/>
 <part name="C14" library="rcl" library_urn="urn:adsk.eagle:library:334" deviceset="C-EU" device="C0201" package3d_urn="urn:adsk.eagle:package:23690/2" value="4.7 uF"/>
@@
 <part name="GND30" library="supply1" library_urn="urn:adsk.eagle:library:371" deviceset="GND" device=""/>
 <part name="GND31" library="SparkFun-Aesthetics" deviceset="GND" device=""/>
+<part name="J2" library="SparkFun-Connectors" deviceset="CONN_02" device="1X02_NO_SILK"/>
 </parts>
 <sheets>
@@
 <attribute name="VALUE" x="316.484" y="74.041" size="1.778" layer="96"/>
 </instance>
-<instance part="C2" gate="G$1" x="38.1" y="33.02" smashed="yes" rot="R180">
-<attribute name="NAME" x="36.576" y="30.099" size="1.778" layer="95" rot="R180"/>
-<attribute name="VALUE" x="36.576" y="37.719" size="1.778" layer="96" rot="R180"/>
-</instance>
 <instance part="C9" gate="G$1" x="48.26" y="33.02" smashed="yes" rot="R180">
 <attribute name="NAME" x="46.736" y="30.099" size="1.778" layer="95" rot="R180"/>
@@
 <attribute name="VALUE" x="64.516" y="37.719" size="1.778" layer="96" rot="R180"/>
 </instance>
-<instance part="GND5" gate="1" x="38.1" y="20.32" smashed="yes">
-<attribute name="VALUE" x="35.56" y="17.78" size="1.778" layer="96"/>
+<instance part="GND5" gate="1" x="48.26" y="20.32" smashed="yes">
+<attribute name="VALUE" x="45.72" y="17.78" size="1.778" layer="96"/>
 </instance>
 <instance part="L3" gate="G$1" x="193.04" y="22.86" smashed="yes">
@@
 <attribute name="VALUE" x="207.899" y="221.234" size="1.778" layer="96" rot="R90"/>
 </instance>
-<instance part="JP2" gate="G$1" x="204.47" y="245.11" smashed="yes">
-<attribute name="NAME" x="201.93" y="247.65" size="1.778" layer="95" font="vector"/>
-</instance>
 <instance part="U$2" gate="G$1" x="226.06" y="33.02" smashed="yes">
 <attribute name="NAME" x="229.108" y="33.02" size="1.778" layer="95" font="vector"/>
@@
 <instance part="GND31" gate="1" x="213.36" y="12.7" smashed="yes">
 <attribute name="VALUE" x="210.82" y="10.16" size="1.778" layer="96"/>
+</instance>
+<instance part="J2" gate="G$1" x="6.35" y="205.74" smashed="yes">
+<attribute name="VALUE" x="3.81" y="200.914" size="1.778" layer="96" font="vector"/>
+<attribute name="NAME" x="3.81" y="211.328" size="1.778" layer="95" font="vector"/>
 </instance>
 </instances>
@@
 </segment>
 <segment>
-<pinref part="C2" gate="G$1" pin="1"/>
 <pinref part="GND5" gate="1" pin="GND"/>
-<wire x1="38.1" y1="22.86" x2="38.1" y2="27.94" width="0.1524" layer="91"/>
 <pinref part="C9" gate="G$1" pin="1"/>
-<wire x1="38.1" y1="27.94" x2="38.1" y2="30.48" width="0.1524" layer="91"/>
 <wire x1="48.26" y1="30.48" x2="48.26" y2="27.94" width="0.1524" layer="91"/>
 <pinref part="C10" gate="G$1" pin="1"/>
 <wire x1="48.26" y1="27.94" x2="55.88" y2="27.94" width="0.1524" layer="91"/>
 <wire x1="55.88" y1="27.94" x2="55.88" y2="30.48" width="0.1524" layer="91"/>
-<wire x1="48.26" y1="27.94" x2="38.1" y2="27.94" width="0.1524" layer="91"/>
+<wire x1="48.26" y1="27.94" x2="48.26" y2="22.86" width="0.1524" layer="91"/>
 <junction x="48.26" y="27.94"/>
-<junction x="38.1" y="27.94"/>
 </segment>
 <segment>
@@
 <label x="170.18" y="50.8" size="1.27" layer="95" xref="yes"/>
 </segment>
+<segment>
+<pinref part="J2" gate="G$1" pin="1"/>
+<wire x1="13.97" y1="205.74" x2="19.05" y2="205.74" width="0.1524" layer="91"/>
+<label x="19.05" y="205.74" size="1.27" layer="95" xref="yes"/>
+</segment>
 </net>
 <net name="TX" class="0">
@@
 <wire x1="162.56" y1="48.26" x2="170.18" y2="48.26" width="0.1524" layer="91"/>
 <label x="170.18" y="48.26" size="1.27" layer="95" xref="yes"/>
+</segment>
+<segment>
+<pinref part="J2" gate="G$1" pin="2"/>
+<wire x1="13.97" y1="208.28" x2="19.05" y2="208.28" width="0.1524" layer="91"/>
+<label x="19.05" y="208.28" size="1.27" layer="95" xref="yes"/>
 </segment>
 </net>
@@
 </segment>
 <segment>
-<pinref part="JP2" gate="G$1" pin="2"/>
-<wire x1="209.55" y1="245.11" x2="214.63" y2="245.11" width="0.1524" layer="91"/>
 <label x="214.63" y="245.11" size="1.27" layer="95" xref="yes"/>
+<pinref part="U4" gate="G$1" pin="BATT"/>
+<wire x1="185.42" y1="245.11" x2="214.63" y2="245.11" width="0.1524" layer="91"/>
 </segment>
 </net>
@@
 <pinref part="C9" gate="G$1" pin="2"/>
 <wire x1="48.26" y1="40.64" x2="48.26" y2="38.1" width="0.1524" layer="91"/>
-<wire x1="48.26" y1="40.64" x2="38.1" y2="40.64" width="0.1524" layer="91"/>
 <junction x="48.26" y="40.64"/>
-<pinref part="C2" gate="G$1" pin="2"/>
-<wire x1="38.1" y1="40.64" x2="38.1" y2="38.1" width="0.1524" layer="91"/>
-<wire x1="38.1" y1="40.64" x2="25.4" y2="40.64" width="0.1524" layer="91"/>
-<junction x="38.1" y="40.64"/>
+<wire x1="48.26" y1="40.64" x2="25.4" y2="40.64" width="0.1524" layer="91"/>
 <label x="25.4" y="40.64" size="1.27" layer="95" rot="R180" xref="yes"/>
 </segment>
@@
 </segment>
 </net>
-<net name="N$10" class="0">
-<segment>
-<pinref part="U4" gate="G$1" pin="BATT"/>
-<wire x1="185.42" y1="245.11" x2="199.39" y2="245.11" width="0.1524" layer="91"/>
-<pinref part="JP2" gate="G$1" pin="1"/>
-</segment>
-</net>
