File: EAGLE/v16/GPS_radiologger_v16.sch (EAGLE design)
At the start: 48 parts, among them IC4 CAT24M01HU5I-GT3, U1 TYPEABZ, U2 UBLOX_ZOE_M8-0-10, U3 MICROCHIP_MCP1810T-33I-J8AMIC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, U4 SPV1050, U5 BME680BME680, Y1 32.768kHz, Y2 W3011

Commit message: recent general edits
Parts:
- removed C12: 10 uF, rcl:C-EUC0201
- removed C6: 0.1 uF, rcl:C-EUC0201
- removed C8: 4.7 uF, rcl:C-EUC0201
- removed JP2: JUMPER-SMT_2_NC_TRACE_NO-SILK, SparkFun-Jumpers:JUMPER-SMT_2_NC_TRACE_NO-SILK
- removed L1: 2.2µH/< 0.2 ohm /500mA, SparkFun-Coils:INDUCTOR-0805-3.3UH
- removed U$5: ALBERT_ZIGZAG-ISP, Zigzag ISP connector:ALBERT_ZIGZAG-ISP
- removed U2: UBLOX_ZOE_M8-0-10, SparkFun-GPS:UBLOX_ZOE_M8-0-10
- removed U3: MICROCHIP_MCP1810T-33I-J8AMICROCHIP_MCP1810T-33I-J8A_0_0, MCP1810:MICROCHIP_MCP1810T-33I-J8AMICROCHIP_MCP1810T-33I-J8A_0_0
- removed Y1: 32.768kHz, SparkFun-Clocks:CRYSTAL-32.768KHZ
- removed Y2: W3011, SparkFun-GPS:GPS_CHIP_ANTENNAW3011
- added J4, J5: (no value), SparkFun-Connectors:CONN_041.27MM_NO_SILK
- added U6: CAM-M8Q-0, CAM-M8Q-0:CAM-M8Q-0
- C13: value 100 uF -> 47 uF
- C2: value 10 uF -> 47 uF
- C5: value 4.7 uF -> 100 nF
- U$3, U$4: value ICARUS_V4_FOOTPRINT -> ICARUS_V4_RAW; device TrisolX_Solar_Cells:ICARUS_V4_FOOTPRINT -> TrisolX_Solar_Cells:ICARUS_V4_RAW
Connections:
- removed net GPS_ANT: U2.RF_IN, Y2.SIGNAL
- removed net N$10: JP2.1, U4.BATT
- removed net N$14: U2.RTC_0, Y1.2
- removed net N$15: U2.RTC_1, Y1.1
- removed net N$3: C5.1, L1.1, U2.V_CORE
- removed net N$5: L1.2, U2.V_DCDC_OUT
- new net N$16: U6.RF_IN, U6.RF_OUT
- net BAT: now also U4.BATT, U4.LDO2_EN; no longer C8.1, JP2.2, U3.!SHDN!, U3.VIN
- net BOOT: now also J5.4; no longer U$5.BOOT
- net GND: now also C2.2, J4.1, U6.GND; no longer C12.2, C2.1, C6.2, C8.2, U$5.GND, U2.GND, U2.SQI_G, U3.GND, U3.GND_PAD, U4.LDO2_EN, Y2.GND
- net POWER: now also J4.2, U4.LDO2, U6.V_BCKP; no longer C12.1, C2.2, U$5.POWER, U2.V_BCKP, U3.FB, U3.VOUT
- net RST: now also J5.1; no longer U$5.RESET
- net RX: now also J4.3
- net SCL: now also U6.SCL/SPI_CLK; no longer U2.SCL/CLK
- net SDA: now also U6.SDA/SPI_CS_N; no longer U2.SDA/CS
- net SWDCLK: now also J5.3; no longer U$5.SWDCLK
- net SWDIO: now also J5.2; no longer U$5.SWDIO
- net TX: now also J4.4
- net ZOE_PWR: now also C2.1, C5.1, U6.VCC, U6.VCC_IO; no longer C6.1, U2.VCC
Other:
- note added: "GNSS/GPS Module CAM-M8Q"
- note removed: "Antenna"
- note removed: "Cut JP2 for battery only operation"
- note removed: "GNSS/GPS Module ZOE-M8Q"
- note removed: "rev14 - add inductor to DC-DC"
- note removed: "rev14 - changed BAT to POWER"
- note removed: "rev14 - tie SQI pins to GND to activate DC-DC pins 29,31,46,47"
- moved on the sheet: C13, C14, C2, C4, C5, PDTA143TMB,1, PDTA143TMB,315, R10, R11, R12, R4, R5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
