File: EAGLE/v16/GPS_radiologger_v16.brd (EAGLE design)
At the start: 40.4 x 26.9 mm, 41 parts, among them IC4 CAT24M01HU5I-GT3, U1 TYPEABZ, U4 SPV1050, U5 BME680BME680, U6 CAM-M8Q-0

Commit message: recent board updates
Parts:
- added C6, C8: (no value), rcl:C0201
- added U2: BMA400, BMA400:XDCR_BMA400
- moved J3 2.58 mm to (4.40, 21.2)
- moved J1 2.09 mm to (7.30, 21.2)
- moved PDTA143TMB,315 0.57 mm to (16.7, 10.9)
- moved R4 0.55 mm to (15.8, 10.9)
- moved PDTA143TMB,1 0.52 mm to (16.8, 9.83)
- moved R5 0.51 mm to (15.9, 9.83)
- moved C14 0.27 mm to (21.1, 14.3)
- moved C3 0.25 mm to (17.4, 5.71)
- moved C13 0.23 mm to (15.8, 13.7)
- moved U$4 0.20 mm to (15.0, 10.8)
- moved J4 0.20 mm to (23.0, 25.0)
- moved J5 0.20 mm to (28.1, 25.0)
- moved C1 0.14 mm to (28.3, 24.1)
Connections:
- new net ACC_INT: U1.P$38, U2.5
- net GND: now also C6.2, C8.2, U2.1, U2.8, U2.9
- net POWER: now also C6.1, C8.1, U2.10, U2.3, U2.7
- net SCL: now also U2.12
- net SDA: now also U2.2
Routing:
- net ACC_INT: track 0.00 -> 23.3 mm, vias 0 -> 2
- net POWER: track 67.3 -> 79.8 mm
- net SCL: track 54.7 -> 60.2 mm, vias 4 -> 5
- net GND: track 150.5 -> 147.3 mm, vias 39 -> 97
- net SDA: track 51.7 -> 53.9 mm
- net N$7: track 33.3 -> 35.4 mm
- net N$11: track 2.84 -> 4.28 mm
- net BAT: track 24.2 -> 25.5 mm
- net RX: track 21.3 -> 20.2 mm
- net N$12: track 7.94 -> 6.90 mm
- net ZOE_PWR: track 20.2 -> 21.2 mm
- net SCD_PWR: track 22.5 -> 23.4 mm
- net VOLT_MEAS: track 22.9 -> 23.5 mm
- net TX: track 24.2 -> 23.6 mm
- net SCD_PDTA: track 18.2 -> 18.8 mm
Other:
- board size 40.4 x 26.9 mm -> 40.4 x 26.1 mm
- board text added: "Max Planck Institute of Animal Behavior Pigeon Pollution Tag v1.16"
- board text removed: "Pollution Tag v1.15.0"
