File: EAGLE/v16/v17/GPS_radiologger_v17.brd (EAGLE design)
At the start: 40.4 x 26.1 mm, 44 parts, among them IC4 CAT24M01HU5I-GT3, U1 TYPEABZ, U2 BMA400, U4 SPV1050, U5 BME680BME680, U6 CAM-M8Q-0

Commit message: recent board updates
Routing:
- net GND: track 147.3 -> 132.7 mm, vias 97 -> 89
- net SDA: track 53.9 -> 46.8 mm
- net SCD_PWR: track 23.4 -> 19.1 mm
- net SCL: track 60.2 -> 58.0 mm
Other:
- board text added: "Max Planck Institute of Animal Behavior Pigeon Pollution Tag v1.16"
- board text removed: "Pollution Tag v1.15.0"
