File: EAGLE/v17/GPS_radiologger_v17.sch (EAGLE design)
At the start: 44 parts, among them IC4 CAT24M01HU5I-GT3, U1 TYPEABZ, U2 BMA400, U4 SPV1050, U5 BME680BME680, U6 CAM-M8Q-0

Commit message: recent board updates
Parts:
- added J2: (no value), SparkFun-Connectors:CONN_041.27MM_NO_SILK
- U$3, U$4: value ICARUS_V4_RAW -> ICARUS_V4_FOOTPRINT; device TrisolX_Solar_Cells:ICARUS_V4_RAW -> TrisolX_Solar_Cells:ICARUS_V4_FOOTPRINT
Connections:
- new net N$18: J4.2
- net DM: now also J4.4
- net DP: now also J4.3
- net POWER: now also J2.1; no longer J4.2
- net RX: now also J2.2; no longer J4.3
- net TX: now also J2.3; no longer J4.4
- net VBUS: now also J2.4
Other:
- moved on the sheet: C13, C14, C4, J4, J5, PDTA143TMB,1, PDTA143TMB,315, R10, R11, R12, R4, R5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
