File: EAGLE/v18_LoRA_only/GPS_radiologger_v18_LoRa_only.brd (EAGLE design)
At the start: 40.4 x 26.1 mm, 44 parts, among them IC4 CAT24M01HU5I-GT3, U1 TYPEABZ, U2 BMA400, U4 SPV1050, U5 BME680BME680, U6 CAM-M8Q-0

Commit message: recent board updates
Parts:
- removed PDTA143TMB,1: TINYPICO-PNPAMB, UnexpectedMaker:SOT883(B)
- removed R5: 100k, rcl:R0201
- removed U$3: ICARUS_V4_RAW, TrisolX_Solar_Cells:ICARUS_FULL_TOP
- added J2: (no value), SparkFun-Connectors:1X04_1.27MM_NO_SILK
- added J6: (no value), SparkFun-Connectors:1X06_1.27MM
- J7: device SparkFun-Connectors:1X07_NO_SILK -> SparkFun-Connectors:1X06_1.27MM
- U$4: value ICARUS_V4_RAW -> ICARUS_V4_FOOTPRINT; device TrisolX_Solar_Cells:ICARUS_FULL_TOP -> TrisolX_Solar_Cells:ICARUS_FULL_FOOTPRINT
- moved R4 13.6 mm to (6.55, 0.91)
- moved R8 13.6 mm to (12.1, 5.05)
- moved U$1 13.5 mm to (10.1, 2.12)
- moved C9 13.5 mm to (11.5, 8.77)
- moved PDTA143TMB,315 13.5 mm to (7.69, 0.89)
- moved C7 13.5 mm to (6.54, 7.87)
- moved C14 13.5 mm to (12.1, 4.23)
- moved C10 13.5 mm to (12.2, 8.77)
- moved C13 13.5 mm to (6.83, 3.70)
- moved R10 13.5 mm to (8.67, 8.07)
- moved R11 13.5 mm to (9.20, 8.64)
- moved R6 13.5 mm to (7.14, 7.87)
- moved U4 13.5 mm to (9.75, 6.02)
- moved R12 13.5 mm to (11.3, 7.93)
- moved R9 13.4 mm to (12.2, 5.79)
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Connections:
- net PWM renamed N$20
- net RDY renamed N$21
- removed net SCD_PWR: J7.7, PDTA143TMB,1.3
- new net N$10: J6.3
- new net N$14: J6.4
- new net N$15: J6.5
- new net N$17: J6.6
- new net N$18: J4.2
- new net N$19: J7.1
- new net N$22: J7.4
- new net N$23: J7.5
- new net N$24: J7.6
- new net N$3: J6.1
- new net N$5: J6.2
- net DM: now also J4.4
- net DP: now also J4.3
- net GND: now also U$4.P$3; no longer J7.1, J7.6, U$3.P$2, U$4.P$2
- net N$7: no longer U$3.P$1
- net POWER: now also J2.1; no longer J4.2, PDTA143TMB,1.2, R5.2
- net RX: now also J2.2; no longer J4.3
- net SCD_PDTA: no longer PDTA143TMB,1.1, R5.1
- net SCL: no longer J7.5
- net SDA: no longer J7.4
- net TX: now also J2.3; no longer J4.4
- net VBUS: now also J2.4
Routing:
- net GND: track 147.3 -> 74.0 mm, vias 97 -> 11
- net SCL: track 60.2 -> 12.2 mm, vias 5 -> 1
- net POWER: track 79.8 -> 33.5 mm
- net SDA: track 53.9 -> 11.3 mm, vias 4 -> 1
- net SCD_PWR: track 23.4 -> 0.00 mm, vias 2 -> 0
- net ACC_INT: track 23.3 -> 3.83 mm, vias 2 -> 1
- net SCD_PDTA: track 18.8 -> 0.00 mm, vias 2 -> 0
- net VOLT_MEAS: track 23.5 -> 5.25 mm, vias 2 -> 1
- net TX: track 23.6 -> 7.09 mm, vias 2 -> 1
- net ZOE_PWR: track 21.2 -> 5.03 mm, vias 2 -> 0
- net N$7: track 35.4 -> 21.2 mm
- net ZOE_PDTA: track 20.6 -> 6.99 mm, vias 2 -> 1
- net RX: track 20.2 -> 8.56 mm, vias 2 -> 1
- net VBUS: track 0.00 -> 9.11 mm, vias 0 -> 1
- net DM: track 0.00 -> 8.22 mm
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Other:
- board size 40.4 x 26.1 mm -> 31.6 x 17 mm
- board text added: "Max Planck Institute of Animal Behavior Pigeon Pollution Tag v1.17"
- board text removed: "Pollution Tag v1.15.0"

Commit message: recent updates
recent updates
Parts:
- removed C11: 0.1uF, rcl:L0201
- removed J4, J5: (no value), SparkFun-Connectors:1X04_1.27MM_NO_SILK
- removed J6, J7: (no value), SparkFun-Connectors:1X06_1.27MM
- removed L3, L4: (no value), rcl:C0201
- removed PDTA143TMB,315: TINYPICO-PNPAMB, UnexpectedMaker:SOT883(B)
- removed R4: 100k, rcl:R0201
- removed U$4: ICARUS_V4_FOOTPRINT, TrisolX_Solar_Cells:ICARUS_FULL_FOOTPRINT
- removed U5: BME680BME680, SparkFun-Sensors:LGA3.0X3.0
- added L2: 2.2uH, SparkFun-Coils:0806
- added U$3, U$5: KXOB25-O5X3F, AnySolar:KXOB25-05X3F
- added U3: BMA400, BMA400:XDCR_BMA400
- added Y1: 32.768kHz, SparkFun-Clocks:CRYSTAL-SMD-3.2X1.5MM
- added Y2: GPS_CHIP_ANTENNAW3011, SparkFun-GPS:W3011
- C2: value 47 uF -> 1 uF
- C3: value 0.1 uF -> (none)
- C5: value 100 nF -> 4.7 uF
- C6: value (none) -> 0.1 uF
- J2: device SparkFun-Connectors:1X04_1.27MM_NO_SILK -> SparkFun-Connectors:1X07_NO_SILK
- U2: value BMA400 -> UBLOX_ZOE_M8-0-10; device BMA400:XDCR_BMA400 -> SparkFun-GPS:UBLOX_ZOE_M8-0-10
- U6: value CAM-M8Q-0 -> TPS22916; device CAM-M8Q-0:LCC100P960X1400X210-31N -> TPS22916V2:TPS22916
- moved C2 18.3 mm to (21.9, 2.50)
- moved R2 16.0 mm to (15.6, 2.05), turned to 0 degrees
- moved U6 15.5 mm to (22.8, 2.00), flipped to the top, turned to 90 degrees
- moved U2 15.1 mm to (6.74, 5.35), flipped to the top, turned to 90 degrees
- moved J2 15.1 mm to (23.9, 16.6)
- moved R1 15.0 mm to (15.6, 1.35), turned to 0 degrees
- moved C6 14.5 mm to (9.43, 3.32), flipped to the top
- moved J3 13.5 mm to (3.50, 1.50)
- moved IC4 12.4 mm to (12.3, 2.40), flipped to the top
- moved C3 10.4 mm to (20.4, 1.20), flipped to the top
- moved C13 7.99 mm to (6.88, 11.7), turned to 90 degrees
- moved C5 6.46 mm to (6.13, 2.44)
- moved J1 5.92 mm to (3.50, 15.1)
- moved U$1 4.72 mm to (13.0, 5.87)
- moved R11 4.70 mm to (11.4, 12.8)
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Connections:
- removed net DM: J4.4, U1.P$2
- removed net DP: J4.3, U1.P$1
- removed net N$10: J6.3
- removed net N$16: U6.16, U6.17
- removed net N$17: J6.6
- removed net N$18: J4.2
- removed net N$19: J7.1
- removed net N$20: J7.2
- removed net N$21: J7.3
- removed net N$22: J7.4
- removed net N$23: J7.5
- removed net N$24: J7.6
- removed net SCD_PDTA: U1.P$23
- removed net VBUS: J2.4, U1.P$20
- removed net ZOE_PDTA: PDTA143TMB,315.1, R4.1, U1.P$24
- removed net ZOE_PWR: C2.1, C5.1, PDTA143TMB,315.3, U6.1, U6.9
- new net GPS_ANT: U2.4, Y2.1
- new net GPS_ON: U1.P$24, U6.B2
- new net GPS_PWR: C6.1, U2.24, U2.25, U6.A1
- new net SAFEBOOT: U1.P$23, U2.34
- net ACC_INT: now also U1.P$21, U3.5; no longer U1.P$38, U2.5
- net BOOT: now also J2.4; no longer J5.4
- net GND: now also J2.5, U$5.P$2, U2.10, U2.11, U2.12, U2.17, U2.23, U2.29, U2.3, U2.31, U2.37, U2.38, U2.39, U2.40, U2.41, U2.44, U2.46, U2.47, U2.49, U2.5, U2.7, U3.1, U3.8, U3.9, U6.B1, Y2.2, Y2.3; no longer J4.1, L3.2, L4.2, U$4.P$3, U5.1, U5.5, U5.7, U6.10, U6.11, U6.12, U6.13, U6.14, U6.15, U6.18, U6.19, U6.21, U6.22, U6.27, U6.31, U6.4, U6.5
- net N$11: now also U1.P$26; no longer C11.1, L4.1
- net N$14: now also U2.18, Y1.P$2; no longer J6.4
- net N$15: now also U2.19, Y1.P$1; no longer J6.5
- net N$2: now also U$3.P$2, U$5.P$1; no longer C11.2, L3.1, U1.P$26
- net N$3: now also L2.2, U2.26; no longer J6.1
- net N$5: now also C5.1, L2.1, U2.27; no longer J6.2
- net N$7: now also U$3.P$1; no longer U$4.P$1
- net POWER: now also C2.1, J2.6, U2.16, U3.10, U3.3, U3.7, U6.A2; no longer C6.1, J2.1, PDTA143TMB,315.2, R4.2, U2.10, U2.3, U2.7, U5.6, U5.8, U6.8
- net RST: now also J2.1; no longer J5.1
- net RX: now also J2.7; no longer J2.2
- net SCL: now also U2.32, U3.12; no longer U2.12, U5.4, U6.6
- net SDA: now also U3.2; no longer U5.3, U6.3
- net SWDCLK: now also J2.3; no longer J5.3
- net SWDIO: now also J2.2; no longer J5.2
- net TX: no longer J2.3
Routing:
- net GND: track 74.0 -> 107.7 mm, vias 11 -> 44
- net SCL: track 12.2 -> 41.8 mm, vias 1 -> 3
- net SDA: track 11.3 -> 40.8 mm, vias 1 -> 4
- net SAFEBOOT: track 0.00 -> 22.2 mm, vias 0 -> 2
- net RX: track 8.56 -> 29.7 mm
- net POWER: track 33.5 -> 54.6 mm, vias 0 -> 7
- net VOLT_MEAS: track 5.25 -> 23.8 mm, vias 1 -> 2
- net GPS_PWR: track 0.00 -> 16.3 mm, vias 0 -> 2
- net VBUS: track 9.11 -> 0.00 mm, vias 1 -> 0
- net DM: track 8.22 -> 0.00 mm
- net N$2: track 1.05 -> 8.81 mm
- net TX: track 7.09 -> 0.00 mm, vias 1 -> 0
- net ZOE_PDTA: track 6.99 -> 0.00 mm, vias 1 -> 0
- net DP: track 5.98 -> 0.00 mm
- net ZOE_PWR: track 5.03 -> 0.00 mm
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- added copper zone on layer 2, net GND
- removed copper zone on layer 16, net GND
Other:
- board size 31.6 x 17 mm -> 33.5 x 16.5 mm
- board text removed: "Max Planck Institute of Animal Behavior Pigeon Pollution Tag v1.17"
