File: EAGLE/v18_LoRA_only/GPS_radiologger_v18_LoRa_only.sch (EAGLE design)
At the start: 44 parts, among them IC4 CAT24M01HU5I-GT3, U1 TYPEABZ, U2 BMA400, U4 SPV1050, U5 BME680BME680, U6 CAM-M8Q-0

Commit message: recent board updates
Parts:
- removed PDTA143TMB,1: TINYPICO-PNPAMB, UnexpectedMaker:TINYPICO-PNPAMB
- removed R5: 100k, rcl:R-EU_R0201
- removed U$3: ICARUS_V4_RAW, TrisolX_Solar_Cells:ICARUS_V4_RAW
- added J2: (no value), SparkFun-Connectors:CONN_041.27MM_NO_SILK
- added J6: (no value), SparkFun-Connectors:CONN_061.27MM
- J7: device SparkFun-Connectors:CONN_07NO_SILK -> SparkFun-Connectors:CONN_061.27MM
- U$4: value ICARUS_V4_RAW -> ICARUS_V4_FOOTPRINT; device TrisolX_Solar_Cells:ICARUS_V4_RAW -> TrisolX_Solar_Cells:ICARUS_V4_FOOTPRINT
Connections:
- net PWM renamed N$20
- net RDY renamed N$21
- removed net SCD_PWR: J7.7, PDTA143TMB,1.C
- new net N$10: J6.3
- new net N$14: J6.4
- new net N$15: J6.5
- new net N$17: J6.6
- new net N$18: J4.2
- new net N$19: J7.1
- new net N$22: J7.4
- new net N$23: J7.5
- new net N$24: J7.6
- new net N$3: J6.1
- new net N$5: J6.2
- net DM: now also J4.4
- net DP: now also J4.3
- net GND: no longer J7.1, J7.6, U$3.MINUS
- net N$7: no longer U$3.PLUS
- net POWER: now also J2.1; no longer J4.2, PDTA143TMB,1.E, R5.2
- net RX: now also J2.2; no longer J4.3
- net SCD_PDTA: no longer PDTA143TMB,1.B, R5.1
- net SCL: no longer J7.5
- net SDA: no longer J7.4
- net TX: now also J2.3; no longer J4.4
- net VBUS: now also J2.4
Other:
- note removed: "CO2 Concentration Sensor Sensirion SCD30"
- note removed: "Default Address 0x61"
- note removed: "Include castellated holes for edge connection"
- note removed: "Pin 1 (SEL) is pulled to GND for I2C operation"
- note removed: "Sensor Power Supply"
- note removed: "future - implement the SGX MICS-2714 Sensor for VOC/NOx"
- moved on the sheet: C13, C14, C4, J4, J5, PDTA143TMB,315, R10, R11, R12, R4, R8, R9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

Commit message: recent updates
recent updates
Parts:
- removed C11: 0.1uF, rcl:L-USL0201
- removed J4, J5: (no value), SparkFun-Connectors:CONN_041.27MM_NO_SILK
- removed J6, J7: (no value), SparkFun-Connectors:CONN_061.27MM
- removed L3, L4: (no value), rcl:C-EUC0201
- removed PDTA143TMB,315: TINYPICO-PNPAMB, UnexpectedMaker:TINYPICO-PNPAMB
- removed R4: 100k, rcl:R-EU_R0201
- removed U$4: ICARUS_V4_FOOTPRINT, TrisolX_Solar_Cells:ICARUS_V4_FOOTPRINT
- removed U5: BME680BME680, SparkFun-Sensors:BME680BME680
- added L2: 2.2uH, SparkFun-Coils:2.2μH_SHIELDED_INDUCTOR
- added U$3, U$5: KXOB25-O5X3F, AnySolar:KXOB25-O5X3F
- added U3: BMA400, BMA400:BMA400
- added Y1: 32.768kHz, SparkFun-Clocks:CRYSTAL-32.768KHZSMD-3.2X1.5
- added Y2: GPS_CHIP_ANTENNAW3011, SparkFun-GPS:GPS_CHIP_ANTENNAW3011
- C2: value 47 uF -> 1 uF
- C3: value 0.1 uF -> (none)
- C5: value 100 nF -> 4.7 uF
- C6: value (none) -> 0.1 uF
- J2: device SparkFun-Connectors:CONN_041.27MM_NO_SILK -> SparkFun-Connectors:CONN_07NO_SILK
- U2: value BMA400 -> UBLOX_ZOE_M8-0-10; device BMA400:BMA400 -> SparkFun-GPS:UBLOX_ZOE_M8-0-10
- U6: value CAM-M8Q-0 -> TPS22916; device CAM-M8Q-0:CAM-M8Q-0 -> TPS22916V2:TPS22916
Connections:
- removed net DM: J4.4, U1.USB_DM
- removed net DP: J4.3, U1.USB_DP
- removed net N$10: J6.3
- removed net N$16: U6.RF_IN, U6.RF_OUT
- removed net N$17: J6.6
- removed net N$18: J4.2
- removed net N$19: J7.1
- removed net N$20: J7.2
- removed net N$21: J7.3
- removed net N$22: J7.4
- removed net N$23: J7.5
- removed net N$24: J7.6
- removed net SCD_PDTA: U1.PA3
- removed net VBUS: J2.4, U1.PA8/MCO
- removed net ZOE_PDTA: PDTA143TMB,315.B, R4.1, U1.PA2
- removed net ZOE_PWR: C2.1, C5.1, PDTA143TMB,315.C, U6.VCC, U6.VCC_IO
- new net GPS_ANT: U2.RF_IN, Y2.SIGNAL
- new net GPS_ON: U1.PA2, U6.ON
- new net GPS_PWR: C6.1, U2.VCC, U6.VOUT
- new net SAFEBOOT: U1.PA3, U2.!SAFEBOOT
- net ACC_INT: now also U1.PA5, U3.INT1; no longer U1.PB7, U2.INT1
- net BOOT: now also J2.4; no longer J5.4
- net GND: now also J2.5, U$5.MINUS, U2.SQI_G, U3.GND, U3.GNDIO, U3.SDO, Y2.GND; no longer J4.1, L3.2, L4.2, U$4.MINUS, U2.GNDIO, U2.SDO, U5.GND, U5.SDO/ADR
- net N$11: now also U1.ANT; no longer C11.1, L4.1
- net N$14: now also U2.RTC_0, Y1.2; no longer J6.4
- net N$15: now also U2.RTC_1, Y1.1; no longer J6.5
- net N$2: now also U$3.MINUS, U$5.PLUS; no longer C11.2, L3.1, U1.ANT
- net N$3: now also L2.2, U2.V_DCDC_OUT; no longer J6.1
- net N$5: now also C5.1, L2.1, U2.V_CORE; no longer J6.2
- net N$7: now also U$3.PLUS; no longer U$4.PLUS
- net POWER: now also C2.1, J2.6, U2.V_BCKP, U3.!CSB, U3.VDD, U3.VDDIO, U6.VIN; no longer C6.1, J2.1, PDTA143TMB,315.E, R4.2, U2.!CSB, U2.VDD, U2.VDDIO, U5.VDD, U5.VDDIO, U6.V_BCKP
- net RST: now also J2.1; no longer J5.1
- net RX: now also J2.7; no longer J2.2
- net SCL: now also U2.SCL/CLK, U3.SCX; no longer U2.SCX, U5.SCK/SCL, U6.SCL/SPI_CLK
- net SDA: now also U2.SDA/CS, U3.SDX; no longer U2.SDX, U5.SDI/SDA, U6.SDA/SPI_CS_N
- net SWDCLK: now also J2.3; no longer J5.3
- net SWDIO: now also J2.2; no longer J5.2
- net TX: no longer J2.3
Other:
- note added: "Coplanar waveguide calculations dielectric (Er) = 4.29 track width (S) = 0.15 mm gap width (W) = 0.101 mm / 4 mil dielectric thickness (h) = 0.08 (b) = 0.352 Effective (Eeff) = 3.167 50.39 Ohms ! Not necessarily ideal, ideally h >> b"
- note added: "GNSS/GPS Module ZOE-M8Q"
- note added: "v18"
- note removed: "Air Quality Sensors"
- note removed: "Coplanar waveguide calculations dielectric (Er) = 4.2 track width (S) = 0.354 gap width (W) = 0.15 dielectric thickness (h) = 0.2 (b) = 0.654 Effective (Eeff) = 2.995 50.02 Ohms ! Not necessarily ideal, ideally h >> b"
- note removed: "Default Address 0x76"
- note removed: "GNSS/GPS Module CAM-M8Q"
- note removed: "General VOC/ RH/ Temp Bosch BME680"
- note removed: "rev14 - add SPV1050 and associated passives"
- note removed: "rev14 - add in zigzag connector for SWD programming"
- note removed: "rev14 - add solar cell"
- note removed: "rev14 - include new antenna land and matching network"
- note removed: "v14"
- moved on the sheet: C13, C14, C2, C3, C4, C5, C6, C8, IC4, R10, R11, R12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
